File: Electrical/BLE_MCU.sch (KiCad schematic (older format))
At the start: 8 parts

Commit message: USB C and RGB IC Schematics
Parts:
- added C5: 0.1uF, symbol Device:C
- added D1: 1N4148, Diode_THT:D_DO-35_SOD27_P7.62mm_Horizontal, symbol Diode:1N4148
- added D2: RED, symbol Device:LED
- added D3: BLUE, symbol Device:LED
- added JP1: Jumper, symbol Device:Jumper
- added R1: 10K, symbol Device:R_US
- added R2, R3: 1K, symbol Device:R_US
- added SW1, SW2: SW_DPST, KMR221:CK-KMR221GLFS-MFG, symbol Switch:SW_DPST
- IC1: renamed from IC?; footprint MDBT42QP512KV2 -> MDBT42Q-P512KV2:MDBT42QP512KV2
- gave numbers to parts that had none: 7
Connections:
- net +3V3: now also D1.1 (K), R1.1
- net DFU: now also SW1.2, SW1.4
- net GND: now also D2.1 (K), D3.1 (K), SW1.1, SW1.3, SW2.2, SW2.4
- net RESET: now also SW2.1, SW2.3
- net at IC1.31 (P0.17): now also R3.1
- net at IC1.33 (P0.19): now also R2.1
- net RX0 renamed RXD
- net TX0 renamed TXD
- new net: C5.2, JP1.1
- new net: D1.2 (A), JP1.2, R1.2
- new net: D3.2 (A), R3.2
- new net: D2.2 (A), R2.2
- new net DTR: C5.1
Other:
- note added: "0.1uF+10K @ 3.3V=\n1.2ms to 0.7VCC"
- moved on the sheet: C1, C2, C3, C4, IC1, L1, L2, Y1
