File: Electrical/Switch_Matrix.sch (KiCad schematic (older format))
At the start: 0 parts

Commit message: USB C and RGB IC Schematics
Parts:
- added C? (x4): 0.47uF, symbol Device:C
- added C? (x3): 0.1uF, symbol Device:C
- added R? (x3): 100k, symbol Device:R_US
- added R?: 20k, symbol Device:R_US
- added R? (x2): 1k, symbol Device:R_US
- added U1: IS31FL3733-TQ, Package_QFP:TQFP-48-1EP_7x7mm_P0.5mm_EP5x5mm, symbol Driver_LED:IS31FL3733-TQ
Connections:
- new net: R?.1, U1.35 (RSET)
- new net: R?.1, U1.47 (IICRST)
- new net +3V3: C?.1, R?.1, R?.1, R?.1, U1.39 (VIO)
- new net GND: C?.1, C?.1, C?.1, C?.1, C?.2, C?.2, C?.2, R?.2, R?.2, R?.2, U1.12 (PGND), U1.34 (AGND), U1.43 (ADDR1), U1.44 (ADDR2), U1.48 (GND), U1.49 (GND), U1.5 (PGND)
- new net INTB: R?.2, U1.45 (~INTB)
- new net SCL: R?.2, U1.42 (SCL)
- new net SDA: R?.2, U1.41 (SDA)
- new net SDB: R?.1, U1.46 (~SDB)
- new net VBUS: C?.1, C?.1, C?.2, C?.2, C?.2, C?.2, U1.20 (PVCC), U1.29 (PVCC), U1.37 (AVCC), U1.38 (DVCC)
- no-connect marks 0 -> 1
